File: board/extended_io.kicad_sch (KiCad schematic)
At the start: 54 parts, among them J5 I2C_3V3, Q10 BC548, Q11 BC548, Q12 BC548, Q13 BC548, Q14 BC548, Q15 BC548, Q16 BC548, Q17 BC548, Q18 BC548, Q7 BC548, Q8 BC548, Q9 BC548, SW11 TD_A, SW12 TD_B, SW13 TD2_A, SW14 TD2_B, SW15 SW_DIP_x03, U10 MCP23008-xP, U11 CAT24C256, U12 MCP7940N-xP, U9 24LC1025, Y1 32.768kHz

Commit message: Do some cleanup after recent changes.
Parts:
- BT1: footprint (none) -> Battery:BatteryHolder_Keystone_1058_1x2032
- J5: footprint (none) -> TerminalBlock_MetzConnect:TerminalBlock_MetzConnect_Type059_RT06304HBWC_1x04_P3.50mm_Horizontal
- SW15: footprint (none) -> Button_Switch_THT:SW_DIP_SPSTx03_Slide_9.78x9.8mm_W7.62mm_P2.54mm
- renumbered C18 to C21, C19 to C22, C20 to C23, C21 to C24, C22 to C25, C23 to C26, D13 to D14, D14 to D15, D15 to D16, D16 to D17, D17 to D18, D18 to D19
Changed lines of the file:
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@@
   (title_block
     (title "The Ulysses Board")
-    (date "2022-09-04")
+    (date "2022-09-08")
     (rev "1.3")
     (company "Dirk Gottschalk")
@@
   (symbol (lib_id "Device:C") (at 236.22 129.54 0) (unit 1)
     (in_bom yes) (on_board yes) (fields_autoplaced)
-    (property "Reference" "C21" (id 0) (at 239.141 128.7053 0)
+    (property "Reference" "C24" (id 0) (at 239.141 128.7053 0)
       (effects (font (size 1.27 1.27)) (justify left))
     )
@@
   (symbol (lib_id "Device:LED") (at 172.72 31.75 90) (unit 1)
     (in_bom yes) (on_board yes) (fields_autoplaced)
-    (property "Reference" "D16" (id 0) (at 175.641 32.5028 90)
+    (property "Reference" "D17" (id 0) (at 175.641 32.5028 90)
       (effects (font (size 1.27 1.27)) (justify right))
     )
@@
     (property "Reference" "SW15" (id 0) (at 105.41 115.6802 0))
     (property "Value" "SW_DIP_x03" (id 1) (at 105.41 118.2171 0))
-    (property "Footprint" "" (id 2) (at 105.41 127 0)
+    (property "Footprint" "Button_Switch_THT:SW_DIP_SPSTx03_Slide_9.78x9.8mm_W7.62mm_P2.54mm" (id 2) (at 105.41 127 0)
       (effects (font (size 1.27 1.27)) hide)
     )
@@
     (property "Reference" "J5" (id 0) (at 139.7 102.9802 90))
     (property "Value" "I2C_3V3" (id 1) (at 139.7 105.5171 90))
-    (property "Footprint" "" (id 2) (at 138.43 107.95 0)
+    (property "Footprint" "TerminalBlock_MetzConnect:TerminalBlock_MetzConnect_Type059_RT06304HBWC_1x04_P3.50mm_Horizontal" (id 2) (at 138.43 107.95 0)
       (effects (font (size 1.27 1.27)) hide)
     )
@@
   (symbol (lib_id "Device:C") (at 17.78 120.65 0) (unit 1)
     (in_bom yes) (on_board yes)
-    (property "Reference" "C18" (id 0) (at 20.701 121.0853 0)
+    (property "Reference" "C21" (id 0) (at 20.701 121.0853 0)
       (effects (font (size 1.27 1.27)) (justify left))
     )
@@
     (property "Reference" "BT1" (id 0) (at 231.648 102.0912 90))
     (property "Value" "CR2032" (id 1) (at 231.648 104.6281 90))
-    (property "Footprint" "" (id 2) (at 232.156 107.95 90)
+    (property "Footprint" "Battery:BatteryHolder_Keystone_1058_1x2032" (id 2) (at 232.156 107.95 90)
       (effects (font (size 1.27 1.27)) hide)
     )
@@
   (symbol (lib_id "Device:LED") (at 119.38 31.75 90) (unit 1)
     (in_bom yes) (on_board yes) (fields_autoplaced)
-    (property "Reference" "D14" (id 0) (at 122.301 32.5028 90)
+    (property "Reference" "D15" (id 0) (at 122.301 32.5028 90)
       (effects (font (size 1.27 1.27)) (justify right))
     )
@@
   (symbol (lib_id "Device:C") (at 254 129.54 0) (unit 1)
     (in_bom yes) (on_board yes) (fields_autoplaced)
-    (property "Reference" "C23" (id 0) (at 256.921 128.7053 0)
+    (property "Reference" "C26" (id 0) (at 256.921 128.7053 0)
       (effects (font (size 1.27 1.27)) (justify left))
     )
@@
   (symbol (lib_id "Device:LED") (at 144.78 31.75 90) (unit 1)
     (in_bom yes) (on_board yes) (fields_autoplaced)
-    (property "Reference" "D15" (id 0) (at 147.701 32.5028 90)
+    (property "Reference" "D16" (id 0) (at 147.701 32.5028 90)
       (effects (font (size 1.27 1.27)) (justify right))
     )
@@
   (symbol (lib_id "Device:LED") (at 203.2 31.75 90) (unit 1)
     (in_bom yes) (on_board yes) (fields_autoplaced)
-    (property "Reference" "D17" (id 0) (at 206.121 32.5028 90)
+    (property "Reference" "D18" (id 0) (at 206.121 32.5028 90)
       (effects (font (size 1.27 1.27)) (justify right))
     )
@@
   (symbol (lib_id "Device:C") (at 92.71 133.35 0) (unit 1)
     (in_bom yes) (on_board yes) (fields_autoplaced)
-    (property "Reference" "C19" (id 0) (at 95.631 132.5153 0)
+    (property "Reference" "C22" (id 0) (at 95.631 132.5153 0)
       (effects (font (size 1.27 1.27)) (justify left))
     )
@@
   (symbol (lib_id "Device:C") (at 248.92 54.61 0) (unit 1)
     (in_bom yes) (on_board yes) (fields_autoplaced)
-    (property "Reference" "C22" (id 0) (at 251.841 53.7753 0)
+    (property "Reference" "C25" (id 0) (at 251.841 53.7753 0)
       (effects (font (size 1.27 1.27)) (justify left))
     )
@@
   (symbol (lib_id "Device:LED") (at 91.44 31.75 90) (unit 1)
     (in_bom yes) (on_board yes) (fields_autoplaced)
-    (property "Reference" "D13" (id 0) (at 94.361 32.5028 90)
+    (property "Reference" "D14" (id 0) (at 94.361 32.5028 90)
       (effects (font (size 1.27 1.27)) (justify right))
     )
@@
   (symbol (lib_id "Device:LED") (at 232.41 31.75 90) (unit 1)
     (in_bom yes) (on_board yes) (fields_autoplaced)
-    (property "Reference" "D18" (id 0) (at 235.331 32.5028 90)
+    (property "Reference" "D19" (id 0) (at 235.331 32.5028 90)
       (effects (font (size 1.27 1.27)) (justify right))
     )
@@
   (symbol (lib_id "Device:C") (at 186.69 121.92 0) (unit 1)
     (in_bom yes) (on_board yes)
-    (property "Reference" "C20" (id 0) (at 189.611 121.0853 0)
-      (effects (font (size 1.27 1.27)) (justify left))
-    )
+    (property "Reference" "C23" (id 0) (at 189.611 121.0853 0)
+      (effects (font (size 1.27 1.27)) (justify left))
+    )
