File: board/ulysses-board.kicad_sch (KiCad schematic)
At the start: 1 part, among them J1 GPIO

Commit message: Fix filenames.
Other:
- sheet Status & I2C module: file untitled.kicad_sch -> extended_io.kicad_sch
Changed lines of the file:
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@@
       (effects (font (size 2 2)) (justify left bottom))
     )
-    (property "Sheet file" "untitled.kicad_sch" (id 1) (at 142.24 117.4246 0)
+    (property "Sheet file" "extended_io.kicad_sch" (id 1) (at 142.24 117.4246 0)
       (effects (font (size 1.27 1.27)) (justify left top) hide)
     )

Commit message: Do some cleanup after recent changes.
Parts:
- J1: footprint Connector_PinSocket_2.54mm:PinSocket_2x20_P2.54mm_Vertical -> Connector_PinHeader_2.54mm:PinHeader_2x20_P2.54mm_Vertical
